Commit message: odom

File: install/sam_bot_description/share/sam_bot_description/src/description/sam_bot_description.urdf (robot description, URDF)
Before this commit: robot sam_bot, 3 links, 2 joints
Links:
- added link imu_link; collision box size=0.1 0.1 0.1; visual box size=0.1 0.1 0.1
- link base_link: geometry collision box size=${base_length} ${base_width} ${base_height}; visual box size=${base_length} ${base_width} ${base_height}
- link front_caster: geometry collision sphere radius=${(wheel_radius+wheel_zoff-(base_height/2))}; visual sphere radius=${(wheel_radius+wheel_zoff-(base_height/2))}
Joints:
- added joint imu_joint: type fixed, parent base_link, child imu_link, origin xyz=0 0 0.01

File: src/description/sam_bot_description.urdf (robot description, URDF)
Before this commit: robot sam_bot, 4 links, 3 joints
Links:
- link base_link: geometry collision box size=${base_length} ${base_width} ${base_height}; visual box size=${base_length} ${base_width} ${base_height}
- link front_caster: geometry collision sphere radius=${(wheel_radius+wheel_zoff-(base_height/2))}; visual sphere radius=${(wheel_radius+wheel_zoff-(base_height/2))}
